Commit message: code update

File: src/abb_with_gripper/urdf/abb_with_measurement_tool.xacro (robot description, xacro)
@@ -5,4 +5,5 @@
   <!-- end-effector -->
   <xacro:include filename="measurement_tool.xacro" />
+  <!-- Camera -->
   <xacro:include filename="$(find realsense2_description)/urdf/_d435.urdf.xacro"/>
   <link name="world" />
@@ -10,4 +11,5 @@
   <!-- end-effector -->
   <xacro:measurement_tool prefix="" connected_to="tool0"/>
+  <!-- Camera -->
   <xacro:arg name="use_nominal_extrinsics" default="True" />
   <xacro:arg name="add_plug" default="false" />
@@ -20,5 +22,5 @@
   <joint name="world_joint" type="fixed">
     <parent link="world" />
-    <child link="base_link" /> <!-- TODO: check base_link name of robot -->
+    <child link="base_link" />
     <origin xyz="0.0 0.0 0.0" rpy="0.0 0.0 0.0" />
   </joint>

File: src/abb_with_gripper/urdf/measurement_tool.xacro (robot description, xacro)
@@ -85,5 +85,5 @@
 <!-- RIGHT FINGER BASE -->
     <joint name="${prefix}finger_right_joint" type="prismatic" >
-      <mimic joint="${prefix}finger_left_joint" multiplier="1" offset="0"/>
+      <!-- <mimic joint="${prefix}finger_left_joint" multiplier="1" offset="0"/> -->
       <parent link="${prefix}measurement_tool" />
       <child link="${prefix}finger_right_link" />
